Commit message: adding a README File to the repository

File: description/gazebo_control.xacro (robot description, xacro)
@@ -6,6 +6,4 @@
             <left_joint>left_wheel_joint</left_joint>
             <right_joint>right_wheel_joint</right_joint>
-            <leftf_joint>leftf_wheel_joint</leftf_joint>
-            <rightf_joint>rightf_wheel_joint</rightf_joint>
             <wheel_separation>0.4</wheel_separation>
             <wheel_diameter>0.1</wheel_diameter>

File: description/robot.urdf.xacro (robot description, xacro)
@@ -3,3 +3,4 @@
     <xacro:include filename="robot_core.xacro" />
     <xacro:include filename="gazebo_control.xacro" />
+    <xacro:include filename="lidar.xacro" />
 </robot>

File: description/robot_core.xacro (robot description, xacro)
@@ -13,4 +13,7 @@
     <material name="black">
         <color rgba="0 0 0 1"/>
+    </material>
+    <material name="red">
+        <color rgba="1 0 0 1"/>
     </material>
     <!-- BASE LINK -->
@@ -70,4 +73,5 @@
         <material>Gazebo/Blue</material>
     </gazebo>
+gazebo_control.
     <!-- LEFT f WHEEL LINK -->
     <joint name="leftf_wheel_joint" type="fixed">
@@ -82,5 +86,5 @@
                 <cylinder radius="0.05" length="0.04"/>
             </geometry>
-            <material name="blue"/>
+            <material name="blue"/>gazebo_control.
         </visual>
         <collision>
