Commit message: adding a README File to the repository

File: description/lidar.xacro (robot description, xacro)
@@ -6,6 +6,6 @@
       <origin xyz="0.2 0 0.125" rpy="0 0 0"/>
    </joint>
-   <link name="laser_frame">
-      <visual>
+ <link name="laser_frame">
+        <visual>
             <geometry>
                 <cylinder radius="0.05" length="0.04"/>
@@ -21,7 +21,7 @@
             <origin xyz="0 0 0" rpy="0 0 0"/>
         </xacro:inertial_cylinder>
-        </link>
+    </link>
     <gazebo reference="laser_frame">
-        <material>Gazebo/Red</material>
+        <material>Gazebo/Black</material>
         <sensor name="laser" type="ray">
             <pose> 0 0 0 0 0 0 </pose>

File: description/robot_core.xacro (robot description, xacro)
@@ -19,4 +19,12 @@
     <!-- BASE LINK -->
     <link name="base_link">
+    </link>
+    <!-- BASE_FOOTPRINT LINK -->
+    <joint name="base_footprint_joint" type="fixed">
+        <parent link="base_link"/>
+        <child link="base_footprint"/>
+        <origin xyz="0 0 0" rpy="0 0 0"/>
+    </joint>
+    <link name="base_footprint">
     </link>
     <!-- CHASSIS LINK -->
